File: FlexCoffeeLED.sch (KiCad schematic (older format))
At the start: 32 parts, among them IC1 NCP718ASN330T1G, IC2 PIC18F25K80-I_SO, IC3 MCP9904T-AE_9Q, J1 Conn_01x05_Male, J2 Conn_01x01_Male, J3 Conn_01x01_Male, Q1 2N3904, Q2 2N3904, Q3 2N3904, U1 PCA9306

Commit message: Created Board Outlines and Keepouts
Parts:
- C1, C10, C2, C3, C4, C5, C6, C7, C8, C9: footprint (none) -> Capacitors_SMD:C_0603
- IC1: footprint SOT95P280X100-5N -> SamacSys_Parts:SOT95P280X100-5N
- IC2: footprint SOIC127P1030X265-28N -> SamacSys_Parts:SOIC127P1030X265-28N
- IC3: footprint SON50P300X300X90-11N-D -> SamacSys_Parts:SON50P300X300X90-11N-D
- J1: footprint (none) -> Pin_Headers:Pin_Header_Straight_1x05_Pitch2.54mm
- J2, J3: footprint (none) -> Pin_Headers:Pin_Header_Straight_1x01_Pitch2.54mm
- JP1: footprint (none) -> LEDs:LED_0603
- Q1, Q2, Q3: footprint Package_TO_SOT_THT:TO-92_Inline -> TO_SOT_Packages_THT:TO-92_Inline_Narrow_Oval
- R1, R2, R3, R4, R5, R6, R7, R8: footprint (none) -> Resistors_SMD:R_0603
- U1: footprint (none) -> SamacSys_Parts:SOP50P310X90-8N
Changed lines of the file:
@@
 F 0 "IC3" H 8700 1915 50  0000 C CNN
 F 1 "MCP9904T-AE_9Q" H 8700 1824 50  0000 C CNN
-F 2 "SON50P300X300X90-11N-D" H 9450 1750 50  0001 L CNN
+F 2 "SamacSys_Parts:SON50P300X300X90-11N-D" H 9450 1750 50  0001 L CNN
 F 3 "https://mouser.componentsearchengine.com/Datasheets/1/MCP9904T-AE_9Q.pdf" H 9450 1650 50  0001 L CNN
 F 4 "Board Mount Temperature Sensors Quad Temp Sensor Addressable Alerts" H 9450 1550 50  0001 L CNN "Description"
@@
 F 0 "IC2" H 4000 4765 50  0000 C CNN
 F 1 "PIC18F25K80-I_SO" H 4000 4674 50  0000 C CNN
-F 2 "SOIC127P1030X265-28N" H 5950 4600 50  0001 L CNN
+F 2 "SamacSys_Parts:SOIC127P1030X265-28N" H 5950 4600 50  0001 L CNN
 F 3 "https://componentsearchengine.com/Datasheets/1/PIC18F25K80-I_SO.pdf" H 5950 4500 50  0001 L CNN
 F 4 "MCU, 32kB Flash,ECAN,12-bit ADC, CTMU" H 5950 4400 50  0001 L CNN "Description"
@@
 F 0 "Q3" H 7140 1496 50  0000 L CNN
 F 1 "2N3904" H 7140 1405 50  0000 L CNN
-F 2 "Package_TO_SOT_THT:TO-92_Inline" H 7150 1375 50  0001 L CIN
+F 2 "TO_SOT_Packages_THT:TO-92_Inline_Narrow_Oval" H 7150 1375 50  0001 L CIN
 F 3 "https://www.fairchildsemi.com/datasheets/2N/2N3904.pdf" H 6950 1450 50  0001 L CNN
 	1    6950 1450
@@
 F 0 "Q1" H 5890 2046 50  0000 L CNN
 F 1 "2N3904" H 5890 1955 50  0000 L CNN
-F 2 "Package_TO_SOT_THT:TO-92_Inline" H 5900 1925 50  0001 L CIN
+F 2 "TO_SOT_Packages_THT:TO-92_Inline_Narrow_Oval" H 5900 1925 50  0001 L CIN
 F 3 "https://www.fairchildsemi.com/datasheets/2N/2N3904.pdf" H 5700 2000 50  0001 L CNN
 	1    5700 2000
@@
 F 0 "Q2" H 6940 2046 50  0000 L CNN
 F 1 "2N3904" H 6940 1955 50  0000 L CNN
-F 2 "Package_TO_SOT_THT:TO-92_Inline" H 6950 1925 50  0001 L CIN
+F 2 "TO_SOT_Packages_THT:TO-92_Inline_Narrow_Oval" H 6950 1925 50  0001 L CIN
 F 3 "https://www.fairchildsemi.com/datasheets/2N/2N3904.pdf" H 6750 2000 50  0001 L CNN
 	1    6750 2000
@@
 F 0 "J1" H 1400 7750 50  0000 C CNN
 F 1 "Conn_01x05_Male" H 1100 7650 50  0000 C CNN
-F 2 "" H 1250 7350 50  0001 C CNN
+F 2 "Pin_Headers:Pin_Header_Straight_1x05_Pitch2.54mm" H 1250 7350 50  0001 C CNN
 F 3 "~" H 1250 7350 50  0001 C CNN
 	1    1250 7350
@@
 F 0 "J3" H 5272 2882 50  0000 R CNN
 F 1 "Conn_01x01_Male" H 5272 2973 50  0000 R CNN
-F 2 "" H 5300 2950 50  0001 C CNN
+F 2 "Pin_Headers:Pin_Header_Straight_1x01_Pitch2.54mm" H 5300 2950 50  0001 C CNN
 F 3 "~" H 5300 2950 50  0001 C CNN
 	1    5300 2950
@@
 F 0 "J2" H 1372 2982 50  0000 R CNN
 F 1 "Conn_01x01_Male" H 1372 3073 50  0000 R CNN
-F 2 "" H 1400 3050 50  0001 C CNN
+F 2 "Pin_Headers:Pin_Header_Straight_1x01_Pitch2.54mm" H 1400 3050 50  0001 C CNN
 F 3 "~" H 1400 3050 50  0001 C CNN
 	1    1400 3050
@@
 F 0 "IC1" H 1950 1465 50  0000 C CNN
 F 1 "NCP718ASN330T1G" H 1950 1374 50  0000 C CNN
-F 2 "SOT95P280X100-5N" H 2400 1300 50  0001 L CNN
+F 2 "SamacSys_Parts:SOT95P280X100-5N" H 2400 1300 50  0001 L CNN
 F 3 "https://componentsearchengine.com/Datasheets/1/NCP718ASN330T1G.pdf" H 2400 1200 50  0001 L CNN
 F 4 "300 MA LOW IQ, WIDE INPUT" H 2400 1100 50  0001 L CNN "Description"
@@
 F 0 "C4" H 2915 1496 50  0000 L CNN
 F 1 "1uF" H 2915 1405 50  0000 L CNN
-F 2 "" H 2838 1300 50  0001 C CNN
+F 2 "Capacitors_SMD:C_0603" H 2838 1300 50  0001 C CNN
 F 3 "~" H 2800 1450 50  0001 C CNN
 	1    2800 1450
@@
 F 0 "C1" H 1015 1346 50  0000 L CNN
 F 1 "1uF" H 1015 1255 50  0000 L CNN
-F 2 "" H 938 1150 50  0001 C CNN
+F 2 "Capacitors_SMD:C_0603" H 938 1150 50  0001 C CNN
 F 3 "~" H 900 1300 50  0001 C CNN
 	1    900  1300
@@
 F 0 "C5" H 3065 3246 50  0000 L CNN
 F 1 "15pF" H 3065 3155 50  0000 L CNN
-F 2 "" H 2988 3050 50  0001 C CNN
+F 2 "Capacitors_SMD:C_0603" H 2988 3050 50  0001 C CNN
 F 3 "~" H 2950 3200 50  0001 C CNN
 	1    2950 3200
@@
 F 0 "C6" H 4165 3246 50  0000 L CNN
 F 1 "15pF" H 4165 3155 50  0000 L CNN
-F 2 "" H 4088 3050 50  0001 C CNN
+F 2 "Capacitors_SMD:C_0603" H 4088 3050 50  0001 C CNN
 F 3 "~" H 4050 3200 50  0001 C CNN
 	1    4050 3200
@@
 F 0 "C3" H 1865 3246 50  0000 L CNN
 F 1 "15pF" H 1865 3155 50  0000 L CNN
-F 2 "" H 1788 3050 50  0001 C CNN
+F 2 "Capacitors_SMD:C_0603" H 1788 3050 50  0001 C CNN
 F 3 "~" H 1750 3200 50  0001 C CNN
 	1    1750 3200
@@
 F 0 "R3" H 7670 5096 50  0000 L CNN
 F 1 "1k" H 7670 5005 50  0000 L CNN
-F 2 "" V 7530 5050 50  0001 C CNN
+F 2 "Resistors_SMD:R_0603" V 7530 5050 50  0001 C CNN
 F 3 "~" H 7600 5050 50  0001 C CNN
 	1    7600 5050
@@
 F 0 "R4" H 7970 5096 50  0000 L CNN
 F 1 "1k" H 7970 5005 50  0000 L CNN
-F 2 "" V 7830 5050 50  0001 C CNN
+F 2 "Resistors_SMD:R_0603" V 7830 5050 50  0001 C CNN
 F 3 "~" H 7900 5050 50  0001 C CNN
 	1    7900 5050
@@
 F 0 "C9" H 6915 5496 50  0000 L CNN
 F 1 "0.1uF" H 6915 5405 50  0000 L CNN
-F 2 "" H 6838 5300 50  0001 C CNN
+F 2 "Capacitors_SMD:C_0603" H 6838 5300 50  0001 C CNN
 F 3 "~" H 6800 5450 50  0001 C CNN
 	1    6800 5450
@@
 F 0 "R1" H 1320 4396 50  0000 L CNN
 F 1 "10k" H 1320 4305 50  0000 L CNN
-F 2 "" V 1180 4350 50  0001 C CNN
+F 2 "Resistors_SMD:R_0603" V 1180 4350 50  0001 C CNN
 F 3 "~" H 1250 4350 50  0001 C CNN
 	1    1250 4350
@@
 F 0 "R2" V 1393 4500 50  0000 C CNN
 F 1 "10k" V 1484 4500 50  0000 C CNN
-F 2 "" V 1530 4500 50  0001 C CNN
+F 2 "Resistors_SMD:R_0603" V 1530 4500 50  0001 C CNN
 F 3 "~" H 1600 4500 50  0001 C CNN
 	1    1600 4500
@@
 F 0 "C2" H 1365 4996 50  0000 L CNN
 F 1 "0.1uF" H 1365 4905 50  0000 L CNN
-F 2 "" H 1288 4800 50  0001 C CNN
+F 2 "Capacitors_SMD:C_0603" H 1288 4800 50  0001 C CNN
 F 3 "~" H 1250 4950 50  0001 C CNN
 	1    1250 4950
@@
 F 0 "JP1" V 1204 4718 50  0000 L CNN
 F 1 "SolderJMOpen" V 1295 4718 50  0000 L CNN
-F 2 "" H 1250 4650 50  0001 C CNN
+F 2 "LEDs:LED_0603" H 1250 4650 50  0001 C CNN
 F 3 "~" H 1250 4650 50  0001 C CNN
 	1    1250 4650
@@
 F 0 "C8" H 6565 1446 50  0000 L CNN
 F 1 "2.2nF" H 6565 1355 50  0000 L CNN
-F 2 "" H 6488 1250 50  0001 C CNN
+F 2 "Capacitors_SMD:C_0603" H 6488 1250 50  0001 C CNN
 F 3 "~" H 6450 1400 50  0001 C CNN
 	1    6450 1400
@@
 F 0 "C7" H 5365 2046 50  0000 L CNN
 F 1 "2.2nF" H 5365 1955 50  0000 L CNN
-F 2 "" H 5288 1850 50  0001 C CNN
+F 2 "Capacitors_SMD:C_0603" H 5288 1850 50  0001 C CNN
 F 3 "~" H 5250 2000 50  0001 C CNN
 	1    5250 2000
@@
 F 0 "U1" H 8800 4561 50  0000 C CNN
 F 1 "PCA9306" H 8800 4470 50  0000 C CNN
-F 2 "" H 8400 5500 50  0001 C CNN
+F 2 "SamacSys_Parts:SOP50P310X90-8N" H 8400 5500 50  0001 C CNN
 F 3 "http://www.ti.com/lit/ds/symlink/pca9306.pdf" H 8500 5600 50  0001 C CNN
 	1    8800 5150
@@
 F 0 "R7" H 9820 5146 50  0000 L CNN
 F 1 "1k" H 9820 5055 50  0000 L CNN
-F 2 "" V 9680 5100 50  0001 C CNN
+F 2 "Resistors_SMD:R_0603" V 9680 5100 50  0001 C CNN
 F 3 "~" H 9750 5100 50  0001 C CNN
 	1    9750 5100
@@
 F 0 "R8" H 10120 5146 50  0000 L CNN
 F 1 "1k" H 10120 5055 50  0000 L CNN
-F 2 "" V 9980 5100 50  0001 C CNN
+F 2 "Resistors_SMD:R_0603" V 9980 5100 50  0001 C CNN
 F 3 "~" H 10050 5100 50  0001 C CNN
 	1    10050 5100
@@
 F 0 "R5" H 8370 4646 50  0000 L CNN
 F 1 "450k" H 8370 4555 50  0000 L CNN
-F 2 "" V 8230 4600 50  0001 C CNN
+F 2 "Resistors_SMD:R_0603" V 8230 4600 50  0001 C CNN
 F 3 "~" H 8300 4600 50  0001 C CNN
 	1    8300 4600
@@
 F 0 "R6" H 9270 4546 50  0000 L CNN
 F 1 "200k" H 9270 4455 50  0000 L CNN
-F 2 "" V 9130 4500 50  0001 C CNN
+F 2 "Resistors_SMD:R_0603" V 9130 4500 50  0001 C CNN
 F 3 "~" H 9200 4500 50  0001 C CNN
 	1    9200 4500
@@
 F 0 "C10" H 9515 4846 50  0000 L CNN
 F 1 "0.1uF" H 9515 4755 50  0000 L CNN
-F 2 "" H 9438 4650 50  0001 C CNN
+F 2 "Capacitors_SMD:C_0603" H 9438 4650 50  0001 C CNN
 F 3 "~" H 9400 4800 50  0001 C CNN
 	1    9400 4800

Commit message: Just Before Renaming Q1 and Q2 Nets
Connections:
- net DN2-DP3 renamed DN2-DP3_N
- net DP2-DN3 renamed DP2-DN3_P
Changed lines of the file:
@@
-$EndComp
-$Comp
-L Transistor_BJT:2N3904 Q3
-U 1 1 5CA36038
-P 6950 1450
-F 0 "Q3" H 7140 1496 50  0000 L CNN
-F 1 "2N3904" H 7140 1405 50  0000 L CNN
-F 2 "TO_SOT_Packages_THT:TO-92_Inline_Narrow_Oval" H 7150 1375 50  0001 L CIN
-F 3 "https://www.fairchildsemi.com/datasheets/2N/2N3904.pdf" H 6950 1450 50  0001 L CNN
-	1    6950 1450
-	1    0    0    -1
 $EndComp
 $Comp
@@
 	5800 2200 6650 2200
 Connection ~ 6650 2200
-Connection ~ 6950 2200
 Wire Wire Line
 	5800 1800 6650 1800
@@
 SDA_5V
 Text Label 6000 1800 0    50   ~ 0
-DP2-DN3
+DP2-DN3_P
 Text Label 6050 2200 0    50   ~ 0
-DN2-DP3
+DN2-DP3_N
 Text Label 7150 1250 0    50   ~ 0
 DP1
@@
 	6450 1250 6750 1250
 Connection ~ 6750 1250
-Wire Wire Line
-	7800 1950 7050 1950
-Wire Wire Line
-	6950 2200 7800 2200
 Wire Wire Line
 	7800 2050 7800 2200
@@
 NoConn ~ 1900 4700
 NoConn ~ 1900 4600
+$Comp
+L Transistor_BJT:2N3904 Q3
+U 1 1 5CA36038
+P 6950 1450
+F 0 "Q3" H 7140 1496 50  0000 L CNN
+F 1 "2N3904" H 7140 1405 50  0000 L CNN
+F 2 "TO_SOT_Packages_THT:TO-92_Inline_Narrow_Oval" H 7150 1375 50  0001 L CIN
+F 3 "https://www.fairchildsemi.com/datasheets/2N/2N3904.pdf" H 6950 1450 50  0001 L CNN
+	1    6950 1450
+	1    0    0    -1
+$EndComp
+Connection ~ 6950 2200
+Wire Wire Line
+	6950 2200 7800 2200
+Wire Wire Line
+	7800 1950 7050 1950
 $EndSCHEMATC

Commit message: First Full Routing of Board
Connections:
- net DN2-DP3_N renamed DN2
- net DP2-DN3_P renamed DP2
Changed lines of the file:
@@
 SDA_5V
 Text Label 6000 1800 0    50   ~ 0
-DP2-DN3_P
+DP2
 Text Label 6050 2200 0    50   ~ 0
-DN2-DP3_N
+DN2
 Text Label 7150 1250 0    50   ~ 0
 DP1

Commit message: A Brand New Design
Parts:
- removed IC1: NCP718ASN330T1G, SamacSys_Parts:SOT95P280X100-5N, symbol SamacSys_Parts:NCP718ASN330T1G
- removed IC2: PIC18F25K80-I_SO, SamacSys_Parts:SOIC127P1030X265-28N, symbol SamacSys_Parts:PIC18F25K80-I_SO
- removed IC3: MCP9904T-AE_9Q, SamacSys_Parts:SON50P300X300X90-11N-D, symbol SamacSys_Parts:MCP9904T-AE_9Q
- removed J2, J3: Conn_01x01_Male, Pin_Headers:Pin_Header_Straight_1x01_Pitch2.54mm, symbol Connector:Conn_01x01_Male
- removed Q1, Q2, Q3: 2N3904, TO_SOT_Packages_THT:TO-92_Inline_Narrow_Oval, symbol Transistor_BJT:2N3904
- removed R5: 450k, Resistors_SMD:R_0603, symbol device:R
- removed R6: 200k, Resistors_SMD:R_0603, symbol device:R
- removed R7, R8: 1k, Resistors_SMD:R_0603, symbol device:R
- removed U1: PCA9306, SamacSys_Parts:SOP50P310X90-8N, symbol interface:PCA9306
- added C11: 0.1uF, Capacitors_SMD:C_0603, symbol device:C
- added IC1, IC3, IC4: LM75BDP,118, SamacSys_Parts:SOP65P490X110-8N, symbol SamacSys_Parts:LM75BDP,118
- added IC2: PIC16F18426-I_ST, SOP65P640X120-14N, symbol SamacSys_Parts:PIC16F18426-I_ST
- added J2, J3: Conn_01x03_Male, Pin_Headers:Pin_Header_Straight_1x03_Pitch2.54mm, symbol Connector:Conn_01x03_Male
- added LED4, LED5, LED6: WS2812B, LEDs:LED_WS2812B-PLCC4, symbol Worldsemi:WS2812B
- C1, C4: value 1uF -> 15pF
- C7: value 2.2nF -> 15pF
- C8: value 2.2nF -> 0.1uF
Connections:
- net DN1 is gone; now on net GND: C8.2
- net DN2 is gone; now on net GND: C7.2
- net DP1 is gone; now on net +5V: C8.1
- net VREF2 is gone; now on net +5V: C10.1
- net +5V: now also R3.1, R4.1, C11.1, IC1.5 (VCC), IC2.1 (VDD), IC3.5 (VCC), IC4.5 (VCC), J2.2 (Pin_2), J3.2 (Pin_2), LED4.1 (VDD), LED5.1 (VDD), LED6.1 (VDD); no longer C1.1
- net GND: now also C11.2, IC1.4 (GND), IC1.6 (A0), IC1.7 (A1), IC1.8 (A2), IC2.14 (VSS), IC3.4 (GND), IC3.7 (A1), IC3.8 (A2), IC4.4 (GND), IC4.6 (A0), IC4.8 (A2), J2.3 (Pin_3), J3.1 (Pin_1), LED4.3 (VSS), LED5.3 (VSS), LED6.3 (VSS); no longer C2.2
- net LED3: now also C1.1; no longer C6.1
- net LED4: now also C4.1, LED4.4 (DIN)
- net MCLR: now also IC2.4 (MCLR/VPP/RA3)
- net PGC: now also IC2.12 (RA1/ICSPCLK)
- net PGD: now also IC2.13 (RA0/ICSPDAT)
- net SCL_5V: now also IC1.2 (SCL), IC2.10 (RC0), IC3.2 (SCL), IC4.2 (SCL)
- net SDA_5V: now also IC1.1 (SDA), IC2.9 (RC1), IC3.1 (SDA), IC4.1 (SDA)
- removed net +3V3: C4.1, R3.1, R4.1
- net DP2 renamed LED6
- net LED6: now also LED5.2 (DOUT), LED6.4 (DIN)
- net LED1 renamed DIN
- net DIN: now also IC2.11 (RA2), J2.1 (Pin_1)
- net SCL_3V: no longer names the net of R4.2
- net SCL_3V: now also IC4.7 (A1)
- net SDA_3V: no longer names the net of R3.2
- net SDA_3V: now also IC3.6 (A0)
- new net DOUT: J3.3 (Pin_3), LED6.2 (DOUT)
- new net LED5: C6.1, LED4.2 (DOUT), LED5.4 (DIN)
- new net SCL2: IC2.5 (RC5)
- new net SDA2: IC2.6 (RC4)
- no-connect marks 22 -> 9
Other:
- note added: "Temperature Sensors"
- note removed: "3V Linear Regulator"
- note removed: "Pull Up Resistors \nAnd Level Converter\nfor I2C Line"
- note removed: "Temperature Sense"
- moved on the sheet: C2, C3, C5, C9, J1, JP1, LED1, LED2, R1, R2
