File: FlexCoffeeLED.kicad_pcb (KiCad board)
At the start: 2 copper layers, 0 parts

Commit message: Created Board Outlines and Keepouts
Parts:
- added C1: 1uF, Capacitors_SMD:C_0603, F.Cu at (232.6, 55.1)
- added C10: 0.1uF, Capacitors_SMD:C_0603, F.Cu at (238.3, 48.2)
- added C2: 0.1uF, Capacitors_SMD:C_0603, F.Cu at (234.5, 51.6)
- added C3: 15pF, Capacitors_SMD:C_0603, F.Cu at (241.7, 45.9)
- added C4: 1uF, Capacitors_SMD:C_0603, F.Cu at (241.7, 43.5)
- added C5: 15pF, Capacitors_SMD:C_0603, F.Cu at (245.6, 41.2)
- added C6: 15pF, Capacitors_SMD:C_0603, F.Cu at (241.7, 41.2)
- added C7: 2.2nF, Capacitors_SMD:C_0603, F.Cu at (246.4, 36.7)
- added C8: 2.2nF, Capacitors_SMD:C_0603, F.Cu at (234.5, 49.3)
- added C9: 0.1uF, Capacitors_SMD:C_0603, F.Cu at (221.5, 58.3)
- added IC1: NCP718ASN330T1G, SamacSys_Parts:SOT95P280X100-5N, F.Cu at (184.0, 91.9)
- added IC2: PIC18F25K80-I_SO, SamacSys_Parts:SOIC127P1030X265-28N, F.Cu at (184.2, 108.2)
- added IC3: MCP9904T-AE_9Q, SamacSys_Parts:SON50P300X300X90-11N-D, F.Cu at (183.9, 96.3)
- added J1: Conn_01x05_Male, Pin_Headers:Pin_Header_Straight_1x05_Pitch2.54mm, F.Cu at (180.0, 96.1)
- added J2: Conn_01x01_Male, Pin_Headers:Pin_Header_Straight_1x01_Pitch2.54mm, F.Cu at (190.4, 52.6)
- added J3: Conn_01x01_Male, Pin_Headers:Pin_Header_Straight_1x01_Pitch2.54mm, F.Cu at (187.7, 40.8)
- added JP1: SolderJMOpen, LEDs:LED_0603, F.Cu at (217.6, 58.3)
- added LED1: WS2812B, LEDs:LED_WS2812B-PLCC4, F.Cu at (182.5, 54.7)
- added LED2: WS2812B, LEDs:LED_WS2812B-PLCC4, F.Cu at (182.5, 46.6)
- added LED3: WS2812B, LEDs:LED_WS2812B-PLCC4, F.Cu at (182.5, 38.6)
- added Q1: 2N3904, TO_SOT_Packages_THT:TO-92_Inline_Narrow_Oval, F.Cu at (189.0, 30.2)
- added Q2: 2N3904, TO_SOT_Packages_THT:TO-92_Inline_Narrow_Oval, F.Cu at (189.4, 85.3)
- added Q3: 2N3904, TO_SOT_Packages_THT:TO-92_Inline_Narrow_Oval, F.Cu at (187.8, 121.2)
- added R1: 10k, Resistors_SMD:R_0603, F.Cu at (245.4, 43.6)
- added R2: 10k, Resistors_SMD:R_0603, F.Cu at (238.2, 50.7)
- added R3: 1k, Resistors_SMD:R_0603, F.Cu at (232.5, 57.5)
- added R4: 1k, Resistors_SMD:R_0603, F.Cu at (242.0, 48.3)
- added R5: 450k, Resistors_SMD:R_0603, F.Cu at (238.2, 53.1)
- added R6: 200k, Resistors_SMD:R_0603, F.Cu at (236.0, 57.5)
- added R7: 1k, Resistors_SMD:R_0603, F.Cu at (241.7, 50.8)
- added R8: 1k, Resistors_SMD:R_0603, F.Cu at (245.6, 46.1)
- added U1: PCA9306, SamacSys_Parts:SOP50P310X90-8N, F.Cu at (181.4, 120.0)
Other:
- board outline added: 12.7 x 97.3 mm
- rule pad_to_mask_clearance: 0.051 -> 0.0762

Commit message: Just Before Renaming Q1 and Q2 Nets
Parts:
- moved C3 93.7 mm to (181.7, 117.9), turned to 180 degrees
- moved Q3 89.0 mm to (189.1, 32.1)
- moved C7 87.9 mm to (183.0, 97.7), turned to 90 degrees
- moved C4 84.3 mm to (180.2, 101.2)
- moved C1 74.7 mm to (179.7, 107.8)
- moved C8 72.8 mm to (180.1, 97.7), turned to 270 degrees
- moved R4 72.3 mm to (180.7, 86.7)
- moved C5 71.6 mm to (181.4, 72.8), turned to 180 degrees
- moved J2 69.0 mm to (179.8, 120.8)
- moved C10 68.5 mm to (178.8, 82.2), turned to 270 degrees
- moved R8 68.1 mm to (179.5, 62.5)
- moved R1 66.7 mm to (179.1, 37.2), turned to 270 degrees
- moved R5 66.3 mm to (179.7, 84.5), turned to 180 degrees
- moved R6 61.2 mm to (178.8, 79.4), turned to 270 degrees
- moved C6 60.5 mm to (181.6, 34.4), turned to 180 degrees
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Connections:
- net /DN2-DP3 renamed /DN2-DP3_N
- net /DP2-DN3 renamed /DP2-DN3_P
Routing:
- net GND: track 0.00 -> 169.1 mm, vias 0 -> 1
- net /DN1: track 0.00 -> 76.2 mm, vias 0 -> 1
- net /DP1: track 0.00 -> 74.6 mm, vias 0 -> 1
- net +5V: track 0.00 -> 5.65 mm
- net /MCLR: track 0.00 -> 5.41 mm
- net /DP2-DN3_P: track 0.00 -> 3.84 mm
- net +3V3: track 0.00 -> 3.67 mm
- net /VREF2: track 0.00 -> 3.38 mm
- net Net-(JP1-Pad1): track 0.00 -> 3.10 mm
- net /LED3: track 0.00 -> 2.16 mm
- net SDA_5V: track 0.00 -> 2.13 mm
- net /DN2-DP3_N: track 0.00 -> 2.13 mm
- net SCL_5V: track 0.00 -> 2.08 mm
- net /PGD: track 0.00 -> 1.88 mm
- net /PGC: track 0.00 -> 1.79 mm
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- added copper zone on F.Cu, net GND
Other:
- net class Default: clearance 0.2 -> 0.1524; trace_width 0.25 -> 0.1778
- net class Diode Pair added: clearance 0.254, trace_width 0.254, via_dia 0.8, via_drill 0.4
- rule trace_clearance: 0.2 -> 0.1524
- rule trace_min: 0.2 -> 0.1778

Commit message: First Full Routing of Board
Parts:
- J1: footprint Pin_Headers:Pin_Header_Straight_1x05_Pitch2.54mm -> BillysCustomLibs:Pin_Header_Straight_1x05_Pitch2.54mm_SMD_Flat
- Q1, Q2, Q3: footprint TO_SOT_Packages_THT:TO-92_Inline_Narrow_Oval -> BillysCustomLibs:TO-92_Inline_Narrow_Oval_SMD
- moved J1 6.87 mm to (188.6, 111.0)
- moved C9 5.34 mm to (186.6, 68.9)
Connections:
- net /DN2-DP3_N renamed /DN2
- net /DP2-DN3_P renamed /DP2
Routing:
- net GND: track 169.1 -> 15.0 mm, vias 1 -> 40
- net +5V: track 5.65 -> 148.5 mm, vias 0 -> 16
- net /LED1: track 0.00 -> 79.5 mm, vias 0 -> 4
- net /PGD: track 1.88 -> 76.6 mm, vias 0 -> 2
- net /PGC: track 1.79 -> 75.7 mm, vias 0 -> 2
- net /MCLR: track 5.41 -> 74.7 mm, vias 0 -> 2
- net /DP2: track 3.84 -> 55.9 mm, vias 0 -> 4
- net /DN2: track 2.13 -> 48.2 mm, vias 0 -> 6
- net /LED2: track 0.00 -> 42.1 mm, vias 0 -> 2
- net /LED3: track 2.16 -> 37.6 mm, vias 0 -> 2
- net SCL_5V: track 2.08 -> 23.8 mm
- net SDA_5V: track 2.13 -> 22.1 mm
- net +3V3: track 3.67 -> 22.3 mm
- net /LED4: track 0.00 -> 11.4 mm
- net SCL_3V: track 0.00 -> 10.3 mm
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- added copper zone on B.Cu, net GND
